Commit message: Imported upstream version '0.1.3' of 'upstream'

File: ridgeback_description/urdf/ridgeback.urdf.xacro (robot description, xacro)
@@ -2,15 +2,13 @@
 <robot name="ridgeback" xmlns:xacro="http://www.ros.org/wiki/xacro">
   <xacro:property name="PI" value="3.1415926535897931" />
-  <xacro:property name="wheelbase" value="0.610" />
-  <xacro:property name="track" value="0.622" />
-  <xacro:property name="wheel_vertical_offset" value="0.05" />
   <xacro:property name="wheel_radius" value="0.0759" />
-  <xacro:property name="wheel_width" value="0.0471" />
-  <xacro:property name="chassis_length" value="0.935" />
-  <xacro:property name="chassis_width" value="0.787" />
+  <xacro:property name="wheel_width" value="0.0790" />
+  <xacro:property name="chassis_length" value="0.960" />
+  <xacro:property name="chassis_width" value="0.793" />
   <xacro:property name="chassis_height" value="0.216" />
+  <xacro:property name="deck_height" value="0.280" />
   <xacro:property name="axle_offset" value="0.0500" />
-  <xacro:property name="rocker_offset" value="0.301525" />
-  <xacro:property name="rocker_width" value="0.568" />
+  <xacro:property name="rocker_offset" value="0.319" />
+  <xacro:property name="rocker_width" value="0.472" />
   <xacro:property name="dummy_inertia" value="1e-09"/>
   <material name="dark_grey"><color rgba="0.2 0.2 0.2 1.0" /></material>
@@ -18,5 +16,5 @@
   <material name="yellow"><color rgba="0.8 0.8 0.0 1.0" /></material>
   <material name="black"><color rgba="0.15 0.15 0.15 1.0" /></material>
-  <xacro:macro name="wheel" params="prefix side y_friction *joint_pose">
+  <xacro:macro name="wheel" params="prefix side *joint_pose">
     <link name="${prefix}_${side}_wheel_link">
       <visual>
@@ -83,9 +81,9 @@
       <xacro:insert_block name="joint_limits" />
     </joint>
-    <xacro:wheel prefix="${prefix}" side="left" y_friction="-0.707107">
+    <xacro:wheel prefix="${prefix}" side="left">
       <origin xyz="0 ${rocker_width/2 + wheel_width/2} 0" rpy="0 0 0" />
     </xacro:wheel>
-    <xacro:wheel prefix="${prefix}" side="right" y_friction="0.707107">
-      <origin xyz="0 ${-rocker_width/2 - wheel_width/2} 0" rpy="0 0 0" />
+    <xacro:wheel prefix="${prefix}" side="right">
+      <origin xyz="0 ${-(rocker_width/2 + wheel_width/2)} 0" rpy="0 0 0" />
     </xacro:wheel>
   </xacro:macro>
@@ -111,5 +109,5 @@
     </visual>
     <collision>
-      <origin xyz="0 0  ${chassis_height/2}"/>
+      <origin xyz="0 0 ${chassis_height/2}"/>
       <geometry>
         <box size="${chassis_length} ${chassis_width} ${chassis_height}"/>
@@ -181,8 +179,4 @@
     </visual>
   </link>
-  <!-- TODO: Make this internal_imu_link or something, and use a mixed-in xacro
-       to supply the joint between it and imu_link. This is important so that imu_link
-       always points to the "active" IMU. When an upgrade IMU is connected, the
-       internal_imu_link should remain, but imu_link should point to the upgrade one. -->
   <link name="imu_link">
     <inertial>
@@ -196,10 +190,16 @@
     <child link="imu_link" />
   </joint>
+  <link name="mid_mount" />
+  <joint name="mid_mount_joint" type="fixed">
+    <parent link="base_link" />
+    <child link="mid_mount" />
+    <origin xyz="0 0 ${deck_height}" rpy="0 0 0"/>
+  </joint>
   <!-- Bring in simulation data for Gazebo. -->
-  <xacro:include filename="ridgeback.gazebo" />
+  <xacro:include filename="$(find ridgeback_description)/urdf/ridgeback.gazebo" />
   <!-- Optional standard accessories, including their simulation data. The rendering
        of these into the final description is controlled by optenv variables, which
        default each one to off.-->
-  <xacro:include filename="accessories.urdf.xacro" />
+  <xacro:include filename="$(find ridgeback_description)/urdf/accessories.urdf.xacro" />
   <!-- Optional custom includes. -->
   <!--<xacro:include filename="$(optenv RIDGEBACK_URDF_EXTRAS empty.urdf)" />-->

Commit message: Imported upstream version '0.1.9' of 'upstream'

File: ridgeback_description/urdf/ridgeback.urdf.xacro (robot description, xacro)
@@ -11,4 +11,7 @@
   <xacro:property name="rocker_offset" value="0.319" />
   <xacro:property name="rocker_width" value="0.472" />
+  <xacro:property name="imu_offset_x" value="0.2085" />
+  <xacro:property name="imu_offset_y" value="-0.2902" />
+  <xacro:property name="imu_offset_z" value="0.1681" />
   <xacro:property name="dummy_inertia" value="1e-09"/>
   <material name="dark_grey"><color rgba="0.2 0.2 0.2 1.0" /></material>
@@ -33,9 +36,9 @@
       <inertial>
         <origin xyz="0 0 0" rpy="0 0 0"/>
-        <mass value="0.477"/>
+        <mass value="2.3"/>
         <inertia
-          ixx="0.0013" ixy="0" ixz="0"
-          iyy="0.0024" iyz="0"
-          izz="0.0013"/>
+          ixx="3.3212e-3" ixy="0" ixz="0"
+          iyy="6.6424e-3" iyz="0"
+          izz="3.3212e-3"/>
       </inertial>
     </link>
@@ -66,10 +69,10 @@
       </visual>
       <inertial>
-        <origin xyz="0 0 0" rpy="0 0 0"/>
-        <mass value="3"/>
+        <origin xyz="0 0 0" rpy="${PI/2} 0 ${PI/2}"/>
+        <mass value="10.267"/>
         <inertia
-          ixx="0.001" ixy="0" ixz="0"
-          iyy="0.001" iyz="0"
-          izz="0.001"/>
+          ixx="0.0288" ixy="2.20484e-6" ixz="-1.3145e-5"
+          iyy="0.4324" iyz="1.8944e-3"
+          izz="0.4130"/>
       </inertial>
     </link>
@@ -102,5 +105,5 @@
   <link name="chassis_link">
     <visual>
-      <origin xyz="0 0 0" rpy=" ${PI/2} 0 ${PI/2}" />
+      <origin xyz="0 0 0" rpy="${PI/2} 0 ${PI/2}" />
       <geometry>
         <mesh filename="package://ridgeback_description/meshes/body.stl"/>
@@ -115,10 +118,10 @@
     </collision>
     <inertial>
-      <origin xyz="0.012 0.002 0.067" rpy="0 0 0"/>
-      <mass value="50"/>
+      <origin xyz="0.012 0.002 0.067" rpy="${PI/2} 0 ${PI/2}"/>
+      <mass value="165.304"/>
       <inertia
-        ixx="1.3136" ixy="0.0" ixz="0.0"
-        iyy="1.3922" iyz="0.0"
-        izz="2.0"/>
+        ixx="4.4744" ixy="0.03098" ixz="0.003647"
+        iyy="7.1624" iyz="0.1228"
+        izz="4.6155"/>
     </inertial>
   </link>
@@ -189,4 +192,5 @@
     <parent link="chassis_link" />
     <child link="imu_link" />
+    <origin xyz="${imu_offset_x} ${imu_offset_y} ${imu_offset_z}" rpy="0 0 0"/>
   </joint>
   <link name="mid_mount" />
